Commit message: tes add parts

File: config/urdf/combined.urdf (robot description, URDF)
Before this commit: robot combined, 17 links, 16 joints
Links:
- added link curve_1_base_link, mass 254.138; visual mesh filename=model://curve_1/meshes/wood.stl scale=0.01 0.01 0.01
- added link curve_2_base_link, mass 254.138; visual mesh filename=model://curve_2/meshes/generic_fan_blade.stl scale=0.01 0.01 0.01
Joints:
- added joint curve_1_pose: type fixed, parent world, child curve_1_base_link, origin xyz=0 0.0 5.0 rpy=0.0 0.0 0.0
- added joint curve_2_pose: type fixed, parent world, child curve_2_base_link, origin xyz=0 0.0 -5.0 rpy=0.0 0.0 0.0

Commit message: add tool

File: config/urdf/combined.urdf (robot description, URDF)
Before this commit: robot combined, 19 links, 18 joints
Links:
- removed link tool0
- added link ABB_6640_180_255_tool; visual mesh filename=model://paintgun/meshes/paint_gun.stl scale=0.04 0.04 0.04
- link curve_1_base_link: geometry visual mesh filename=model://curve_1/meshes/wood.stl scale=0.05 0.05 0.05
- link curve_2_base_link: geometry visual mesh filename=model://curve_2/meshes/generic_fan_blade.stl scale=0.05 0.05 0.05
Joints:
- joint curve_1_pose: origin xyz=0 0.0 5.0 rpy=0.0 0.0 0.0 -> xyz=0 2.0 0.0 rpy=0.0 0.0 0.0
- joint curve_2_pose: origin xyz=0 0.0 -5.0 rpy=0.0 0.0 0.0 -> xyz=0 -2.0 0.0 rpy=0.0 0.0 0.0
- joint joint_6-tool0: child tool0 -> ABB_6640_180_255_tool

Commit message: tes scale

File: config/urdf/combined.urdf (robot description, URDF)
Before this commit: robot combined, 19 links, 18 joints
Links:
- removed link abb_1200_5_90_pedestal
- added link ABB_1200_5_90_pedestal, mass 1; visual cylinder length=1.0 radius=0.2
- added link FANUC_lrmate200id_base_link; collision mesh filename=model://FANUC_lrmate200id/meshes/lrmate200id/collision/base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; visual mesh filename=model://FANUC_lrmate200id/meshes/lrmate200id/visual/base_li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
- added link FANUC_lrmate200id_link_1; collision mesh filename=model://FANUC_lrmate200id/meshes/lrmate200id/collision/link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; visual mesh filename=model://FANUC_lrmate200id/meshes/lrmate200id/visual/link_1.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
- added link FANUC_lrmate200id_link_2; collision mesh filename=model://FANUC_lrmate200id/meshes/lrmate200id/collision/link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; visual mesh filename=model://FANUC_lrmate200id/meshes/lrmate200id/visual/link_2.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
- added link FANUC_lrmate200id_link_3; collision mesh filename=model://FANUC_lrmate200id/meshes/lrmate200id/collision/link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; visual mesh filename=model://FANUC_lrmate200id/meshes/lrmate200id/visual/link_3.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
- added link FANUC_lrmate200id_link_4; collision mesh filename=model://FANUC_lrmate200id/meshes/lrmate200id/collision/link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; visual mesh filename=model://FANUC_lrmate200id/meshes/lrmate200id/visual/link_4.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
- added link FANUC_lrmate200id_link_5; collision mesh filename=model://FANUC_lrmate200id/meshes/lrmate200id/collision/link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; visual mesh filename=model://FANUC_lrmate200id/meshes/lrmate200id/visual/link_5.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
- added link FANUC_lrmate200id_link_6; collision mesh filename=model://FANUC_lrmate200id/meshes/lrmate200id/collision/link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; visual mesh filename=model://FANUC_lrmate200id/meshes/lrmate200id/visual/link_6.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
- added link FANUC_m10ia_base_link; collision mesh filename=model://FANUC_m10ia/meshes/m10ia/collision/base_link.stl; visual mesh filename=model://FANUC_m10ia/meshes/m10ia/visual/base_link.stl
- added link FANUC_m10ia_link_1; collision mesh filename=model://FANUC_m10ia/meshes/m10ia/collision/link_1.stl; visual mesh filename=model://FANUC_m10ia/meshes/m10ia/visual/link_1.stl
- added link FANUC_m10ia_link_2; collision mesh filename=model://FANUC_m10ia/meshes/m10ia/collision/link_2.stl; visual mesh filename=model://FANUC_m10ia/meshes/m10ia/visual/link_2.stl
- added link FANUC_m10ia_link_3; collision mesh filename=model://FANUC_m10ia/meshes/m10ia/collision/link_3.stl; visual mesh filename=model://FANUC_m10ia/meshes/m10ia/visual/link_3.stl
- added link FANUC_m10ia_link_4; collision mesh filename=model://FANUC_m10ia/meshes/m10ia/collision/link_4.stl; visual mesh filename=model://FANUC_m10ia/meshes/m10ia/visual/link_4.stl
- added link FANUC_m10ia_link_5; collision mesh filename=model://FANUC_m10ia/meshes/m10ia/collision/link_5.stl; visual mesh filename=model://FANUC_m10ia/meshes/m10ia/visual/link_5.stl
- added link FANUC_m10ia_link_6; collision mesh filename=model://FANUC_m10ia/meshes/m10ia/collision/link_6.stl; visual mesh filename=model://FANUC_m10ia/meshes/m10ia/visual/link_6.stl
- added link FANUC_m10ia_tool; visual mesh filename=model://paintgun/meshes/paint_gun.stl scale=0.001 0.001 0.001
- link ABB_1200_5_90_base_link: geometry visual mesh filename=model://ABB_1200_5_90/meshes/visual/base_link.dae scale=1 1 1
- link ABB_1200_5_90_link_1: geometry collision mesh filename=model://ABB_1200_5_90/meshes/collision/link_1.stl scale=1 1 1; visual mesh filename=model://ABB_1200_5_90/meshes/visual/link_1.dae scale=1 1 1
- link ABB_1200_5_90_link_2: geometry collision mesh filename=model://ABB_1200_5_90/meshes/collision/link_2.stl scale=1 1 1; visual mesh filename=model://ABB_1200_5_90/meshes/visual/link_2.dae scale=1 1 1
- link ABB_1200_5_90_link_3: geometry collision mesh filename=model://ABB_1200_5_90/meshes/collision/link_3.stl scale=1 1 1; visual mesh filename=model://ABB_1200_5_90/meshes/visual/link_3.dae scale=1 1 1
- link ABB_1200_5_90_link_4: geometry collision mesh filename=model://ABB_1200_5_90/meshes/collision/link_4.stl scale=1 1 1; visual mesh filename=model://ABB_1200_5_90/meshes/visual/link_4.dae scale=1 1 1
- link ABB_1200_5_90_link_5: geometry collision mesh filename=model://ABB_1200_5_90/meshes/collision/link_5.stl scale=1 1 1; visual mesh filename=model://ABB_1200_5_90/meshes/visual/link_5.dae scale=1 1 1
- link ABB_1200_5_90_link_6: geometry collision mesh filename=model://ABB_1200_5_90/meshes/collision/link_6.stl scale=1 1 1; visual mesh filename=model://ABB_1200_5_90/meshes/visual/link_6.dae scale=1 1 1
- link ABB_6640_180_255_base_link: geometry collision box size=1.016 .729 .24; visual mesh filename=model://ABB_6640_180_255/meshes/visual/Base.stl
- link ABB_6640_180_255_link_1: geometry collision box size=.31 .528 .368; collision box size=.436 .328 .192
- link ABB_6640_180_255_link_2: geometry collision box size=.251 .169 .058; collision box size=.538 1.429 .311
- link ABB_6640_180_255_link_3: geometry collision box size=.052 .085 .102; collision box size=.052 .109 .102
- link ABB_6640_180_255_link_4: geometry collision box size=.145 .278 .075; collision box size=.145 .278 .092
- link ABB_6640_180_255_link_5: geometry collision cylinder length=.307 radius=.107; visual mesh filename=model://ABB_6640_180_255/meshes/visual/Link5.stl
- link ABB_6640_180_255_link_6: geometry collision cylinder length=.037 radius=.109; visual mesh filename=model://ABB_6640_180_255/meshes/visual/Link6.stl
- link ABB_6640_180_255_tool: geometry visual mesh filename=model://paintgun/meshes/paint_gun.stl scale=0.001 0.001 0.001
- link curve_1_base_link: geometry visual mesh filename=model://curve_1/meshes/wood.stl scale=0.001 0.001 0.001
- link curve_2_base_link: geometry visual mesh filename=model://curve_2/meshes/generic_fan_blade.stl scale=0.001 0.001 0.001
Joints:
- removed joint abb_1200_5_90_pedestal_JOINT_0
- removed joint abb_1200_5_90_pose
- removed joint abb_6640_180_255_pose
- added joint ABB_1200_5_90_pedestal_JOINT_0: type fixed, parent ABB_1200_5_90_pedestal, child ABB_1200_5_90_base_link, origin xyz=0 0 0 rpy=0 0 0, axis 0 0 0, limit lower=0 upper=0 effort=0 velocity=0
- added joint ABB_1200_5_90_pose: type fixed, parent world, child ABB_1200_5_90_pedestal, origin xyz=0 5.0 5.0 rpy=0.0 0.0 0.0
- added joint ABB_6640_180_255_pose: type fixed, parent world, child ABB_6640_180_255_base_link, origin xyz=0 0 0.0 rpy=0.0 0.0 0.0
- added joint FANUC_lrmate200id_joint_1: type revolute, parent FANUC_lrmate200id_base_link, child FANUC_lrmate200id_link_1, origin xyz=0 0 0.330 rpy=0 0 0, axis 0 0 1, limit lower=-2.9670597283903604 upper=2.9670597283903604 effort=0 velocity=7.853981633974483
- added joint FANUC_lrmate200id_joint_2: type revolute, parent FANUC_lrmate200id_link_1, child FANUC_lrmate200id_link_2, origin xyz=0.050 0 0 rpy=0 0 0, axis 0 1 0, limit lower=-1.7453292519943295 upper=2.530727415391778 effort=0 velocity=6.632251157578453
- added joint FANUC_lrmate200id_joint_3: type revolute, parent FANUC_lrmate200id_link_2, child FANUC_lrmate200id_link_3, origin xyz=0 0 0.330 rpy=0 0 0, axis 0 -1 0, limit lower=-1.2217304763960306 upper=3.5779249665883754 effort=0 velocity=9.075712110370514
- added joint FANUC_lrmate200id_joint_4: type revolute, parent FANUC_lrmate200id_link_3, child FANUC_lrmate200id_link_4, origin xyz=0 0 0.035 rpy=0 0 0, axis -1 0 0, limit lower=-3.3161255787892263 upper=3.3161255787892263 effort=0 velocity=9.599310885968812
- added joint FANUC_lrmate200id_joint_5: type revolute, parent FANUC_lrmate200id_link_4, child FANUC_lrmate200id_link_5, origin xyz=0.335 0 0 rpy=0 0 0, axis 0 -1 0, limit lower=-2.181661564992912 upper=2.181661564992912 effort=0 velocity=9.512044423369096
- added joint FANUC_lrmate200id_joint_6: type revolute, parent FANUC_lrmate200id_link_5, child FANUC_lrmate200id_link_6, origin xyz=0.080 0 0 rpy=0 0 0, axis -1 0 0, limit lower=-6.283185307179586 upper=6.283185307179586 effort=0 velocity=17.453292519943297
- added joint FANUC_lrmate200id_pose: type fixed, parent world, child FANUC_lrmate200id_base_link, origin xyz=0 -5.0 5.0 rpy=0.0 0.0 0.0
- added joint FANUC_m10ia_joint_1: type revolute, parent FANUC_m10ia_base_link, child FANUC_m10ia_link_1, origin xyz=0 0 0.450 rpy=0 0 0, axis 0 0 1, limit lower=-3.14 upper=3.14 effort=0 velocity=3.67
- added joint FANUC_m10ia_joint_2: type revolute, parent FANUC_m10ia_link_1, child FANUC_m10ia_link_2, origin xyz=0.150 0 0 rpy=0 0 0, axis 0 1 0, limit lower=-1.57 upper=2.79 effort=0 velocity=3.32
- added joint FANUC_m10ia_joint_3: type revolute, parent FANUC_m10ia_link_2, child FANUC_m10ia_link_3, origin xyz=0 0 0.600 rpy=0 0 0, axis 0 -1 0, limit lower=-3.14 upper=4.61 effort=0 velocity=3.67
- added joint FANUC_m10ia_joint_4: type revolute, parent FANUC_m10ia_link_3, child FANUC_m10ia_link_4, origin xyz=0 0 0.200 rpy=0 0 0, axis -1 0 0, limit lower=-3.31 upper=3.31 effort=0 velocity=6.98
- added joint FANUC_m10ia_joint_5: type revolute, parent FANUC_m10ia_link_4, child FANUC_m10ia_link_5, origin xyz=0.640 0 0 rpy=0 0 0, axis 0 -1 0, limit lower=-3.31 upper=3.31 effort=0 velocity=6.98
- added joint FANUC_m10ia_joint_6: type revolute, parent FANUC_m10ia_link_5, child FANUC_m10ia_link_6, origin xyz=0.100 0 0 rpy=0 0 0, axis -1 0 0, limit lower=-6.28 upper=6.28 effort=0 velocity=10.47
- added joint FANUC_m10ia_joint_6-tool0: type fixed, parent FANUC_m10ia_link_6, child FANUC_m10ia_tool, origin xyz=0 0 0 rpy=0 1.57079632679 0
- added joint FANUC_m10ia_pose: type fixed, parent world, child FANUC_m10ia_base_link, origin xyz=0 0.0 5.0 rpy=0.0 0.0 0.0

Commit message: diffevo with collision

File: config/urdf/combined.urdf (robot description, URDF)
Before this commit: robot combined, 34 links, 33 joints
Links:
- link ABB_6640_180_255_tool: geometry collision mesh filename=model://paintgun/meshes/paint_gun.stl scale=0.001 0.001 0.001; visual mesh filename=model://paintgun/meshes/paint_gun.stl scale=0.001 0.001 0.001
- link FANUC_m10ia_tool: geometry collision mesh filename=model://paintgun/meshes/paint_gun.stl scale=0.001 0.001 0.001; visual mesh filename=model://paintgun/meshes/paint_gun.stl scale=0.001 0.001 0.001
- link curve_1_base_link: geometry collision mesh filename=model://curve_1/meshes/wood.stl scale=0.001 0.001 0.001; visual mesh filename=model://curve_1/meshes/wood.stl scale=0.001 0.001 0.001
- link curve_2_base_link: geometry collision mesh filename=model://curve_2/meshes/generic_fan_blade.stl scale=0.001 0.001 0.001; visual mesh filename=model://curve_2/meshes/generic_fan_blade.stl scale=0.001 0.001 0.001
Joints:
- joint ABB_6640_180_255_pose: origin xyz=0 0 0.0 rpy=0.0 0.0 0.0 -> xyz=5.0 0 5.0 rpy=0.0 0.0 0.0

Commit message: update from main

File: config/urdf/combined.urdf (robot description, URDF)
Before this commit: robot combined, 19 links, 18 joints
Links:
- removed link abb_1200_5_90_pedestal
- removed link tool0
- added link ABB_1200_5_90_pedestal, mass 1; visual cylinder length=1.0 radius=0.2
- added link ABB_6640_180_255_tool; collision mesh filename=model://paintgun/meshes/paint_gun.stl scale=0.001 0.001 0.001; visual mesh filename=model://paintgun/meshes/paint_gun.stl scale=0.001 0.001 0.001
- added link FANUC_lrmate200id_base_link; collision mesh filename=model://FANUC_lrmate200id/meshes/lrmate200id/collision/base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; visual mesh filename=model://FANUC_lrmate200id/meshes/lrmate200id/visual/base_li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
- added link FANUC_lrmate200id_link_1; collision mesh filename=model://FANUC_lrmate200id/meshes/lrmate200id/collision/link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; visual mesh filename=model://FANUC_lrmate200id/meshes/lrmate200id/visual/link_1.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
- added link FANUC_lrmate200id_link_2; collision mesh filename=model://FANUC_lrmate200id/meshes/lrmate200id/collision/link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; visual mesh filename=model://FANUC_lrmate200id/meshes/lrmate200id/visual/link_2.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
- added link FANUC_lrmate200id_link_3; collision mesh filename=model://FANUC_lrmate200id/meshes/lrmate200id/collision/link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; visual mesh filename=model://FANUC_lrmate200id/meshes/lrmate200id/visual/link_3.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
- added link FANUC_lrmate200id_link_4; collision mesh filename=model://FANUC_lrmate200id/meshes/lrmate200id/collision/link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; visual mesh filename=model://FANUC_lrmate200id/meshes/lrmate200id/visual/link_4.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
- added link FANUC_lrmate200id_link_5; collision mesh filename=model://FANUC_lrmate200id/meshes/lrmate200id/collision/link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; visual mesh filename=model://FANUC_lrmate200id/meshes/lrmate200id/visual/link_5.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
- added link FANUC_lrmate200id_link_6; collision mesh filename=model://FANUC_lrmate200id/meshes/lrmate200id/collision/link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; visual mesh filename=model://FANUC_lrmate200id/meshes/lrmate200id/visual/link_6.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
- added link FANUC_m10ia_base_link; collision mesh filename=model://FANUC_m10ia/meshes/m10ia/collision/base_link.stl; visual mesh filename=model://FANUC_m10ia/meshes/m10ia/visual/base_link.stl
- added link FANUC_m10ia_link_1; collision mesh filename=model://FANUC_m10ia/meshes/m10ia/collision/link_1.stl; visual mesh filename=model://FANUC_m10ia/meshes/m10ia/visual/link_1.stl
- added link FANUC_m10ia_link_2; collision mesh filename=model://FANUC_m10ia/meshes/m10ia/collision/link_2.stl; visual mesh filename=model://FANUC_m10ia/meshes/m10ia/visual/link_2.stl
- added link FANUC_m10ia_link_3; collision mesh filename=model://FANUC_m10ia/meshes/m10ia/collision/link_3.stl; visual mesh filename=model://FANUC_m10ia/meshes/m10ia/visual/link_3.stl
- added link FANUC_m10ia_link_4; collision mesh filename=model://FANUC_m10ia/meshes/m10ia/collision/link_4.stl; visual mesh filename=model://FANUC_m10ia/meshes/m10ia/visual/link_4.stl
- added link FANUC_m10ia_link_5; collision mesh filename=model://FANUC_m10ia/meshes/m10ia/collision/link_5.stl; visual mesh filename=model://FANUC_m10ia/meshes/m10ia/visual/link_5.stl
- added link FANUC_m10ia_link_6; collision mesh filename=model://FANUC_m10ia/meshes/m10ia/collision/link_6.stl; visual mesh filename=model://FANUC_m10ia/meshes/m10ia/visual/link_6.stl
- added link FANUC_m10ia_tool; collision mesh filename=model://paintgun/meshes/paint_gun.stl scale=0.001 0.001 0.001; visual mesh filename=model://paintgun/meshes/paint_gun.stl scale=0.001 0.001 0.001
- link ABB_1200_5_90_base_link: geometry visual mesh filename=model://ABB_1200_5_90/meshes/visual/base_link.dae scale=1 1 1
- link ABB_1200_5_90_link_1: geometry collision mesh filename=model://ABB_1200_5_90/meshes/collision/link_1.stl scale=1 1 1; visual mesh filename=model://ABB_1200_5_90/meshes/visual/link_1.dae scale=1 1 1
- link ABB_1200_5_90_link_2: geometry collision mesh filename=model://ABB_1200_5_90/meshes/collision/link_2.stl scale=1 1 1; visual mesh filename=model://ABB_1200_5_90/meshes/visual/link_2.dae scale=1 1 1
- link ABB_1200_5_90_link_3: geometry collision mesh filename=model://ABB_1200_5_90/meshes/collision/link_3.stl scale=1 1 1; visual mesh filename=model://ABB_1200_5_90/meshes/visual/link_3.dae scale=1 1 1
- link ABB_1200_5_90_link_4: geometry collision mesh filename=model://ABB_1200_5_90/meshes/collision/link_4.stl scale=1 1 1; visual mesh filename=model://ABB_1200_5_90/meshes/visual/link_4.dae scale=1 1 1
- link ABB_1200_5_90_link_5: geometry collision mesh filename=model://ABB_1200_5_90/meshes/collision/link_5.stl scale=1 1 1; visual mesh filename=model://ABB_1200_5_90/meshes/visual/link_5.dae scale=1 1 1
- link ABB_1200_5_90_link_6: geometry collision mesh filename=model://ABB_1200_5_90/meshes/collision/link_6.stl scale=1 1 1; visual mesh filename=model://ABB_1200_5_90/meshes/visual/link_6.dae scale=1 1 1
- link ABB_6640_180_255_base_link: geometry collision box size=1.016 .729 .24; visual mesh filename=model://ABB_6640_180_255/meshes/visual/Base.stl
- link ABB_6640_180_255_link_1: geometry collision box size=.31 .528 .368; collision box size=.436 .328 .192
- link ABB_6640_180_255_link_2: geometry collision box size=.251 .169 .058; collision box size=.538 1.429 .311
- link ABB_6640_180_255_link_3: geometry collision box size=.052 .085 .102; collision box size=.052 .109 .102
- link ABB_6640_180_255_link_4: geometry collision box size=.145 .278 .075; collision box size=.145 .278 .092
- link ABB_6640_180_255_link_5: geometry collision cylinder length=.307 radius=.107; visual mesh filename=model://ABB_6640_180_255/meshes/visual/Link5.stl
- link ABB_6640_180_255_link_6: geometry collision cylinder length=.037 radius=.109; visual mesh filename=model://ABB_6640_180_255/meshes/visual/Link6.stl
- link curve_1_base_link: geometry collision mesh filename=model://curve_1/meshes/wood.stl scale=0.001 0.001 0.001; visual mesh filename=model://curve_1/meshes/wood.stl scale=0.001 0.001 0.001
- link curve_2_base_link: geometry collision mesh filename=model://curve_2/meshes/generic_fan_blade.stl scale=0.001 0.001 0.001; visual mesh filename=model://curve_2/meshes/generic_fan_blade.stl scale=0.001 0.001 0.001
Joints:
- removed joint abb_1200_5_90_pedestal_JOINT_0
- removed joint abb_1200_5_90_pose
- removed joint abb_6640_180_255_pose
- added joint ABB_1200_5_90_pedestal_JOINT_0: type fixed, parent ABB_1200_5_90_pedestal, child ABB_1200_5_90_base_link, origin xyz=0 0 0 rpy=0 0 0, axis 0 0 0, limit lower=0 upper=0 effort=0 velocity=0
- added joint ABB_1200_5_90_pose: type fixed, parent world, child ABB_1200_5_90_pedestal, origin xyz=0 5.0 5.0 rpy=0.0 0.0 0.0
- added joint ABB_6640_180_255_pose: type fixed, parent world, child ABB_6640_180_255_base_link, origin xyz=5.0 0 5.0 rpy=0.0 0.0 0.0
- added joint FANUC_lrmate200id_joint_1: type revolute, parent FANUC_lrmate200id_base_link, child FANUC_lrmate200id_link_1, origin xyz=0 0 0.330 rpy=0 0 0, axis 0 0 1, limit lower=-2.9670597283903604 upper=2.9670597283903604 effort=0 velocity=7.853981633974483
- added joint FANUC_lrmate200id_joint_2: type revolute, parent FANUC_lrmate200id_link_1, child FANUC_lrmate200id_link_2, origin xyz=0.050 0 0 rpy=0 0 0, axis 0 1 0, limit lower=-1.7453292519943295 upper=2.530727415391778 effort=0 velocity=6.632251157578453
- added joint FANUC_lrmate200id_joint_3: type revolute, parent FANUC_lrmate200id_link_2, child FANUC_lrmate200id_link_3, origin xyz=0 0 0.330 rpy=0 0 0, axis 0 -1 0, limit lower=-1.2217304763960306 upper=3.5779249665883754 effort=0 velocity=9.075712110370514
- added joint FANUC_lrmate200id_joint_4: type revolute, parent FANUC_lrmate200id_link_3, child FANUC_lrmate200id_link_4, origin xyz=0 0 0.035 rpy=0 0 0, axis -1 0 0, limit lower=-3.3161255787892263 upper=3.3161255787892263 effort=0 velocity=9.599310885968812
- added joint FANUC_lrmate200id_joint_5: type revolute, parent FANUC_lrmate200id_link_4, child FANUC_lrmate200id_link_5, origin xyz=0.335 0 0 rpy=0 0 0, axis 0 -1 0, limit lower=-2.181661564992912 upper=2.181661564992912 effort=0 velocity=9.512044423369096
- added joint FANUC_lrmate200id_joint_6: type revolute, parent FANUC_lrmate200id_link_5, child FANUC_lrmate200id_link_6, origin xyz=0.080 0 0 rpy=0 0 0, axis -1 0 0, limit lower=-6.283185307179586 upper=6.283185307179586 effort=0 velocity=17.453292519943297
- added joint FANUC_lrmate200id_pose: type fixed, parent world, child FANUC_lrmate200id_base_link, origin xyz=0 -5.0 5.0 rpy=0.0 0.0 0.0
- added joint FANUC_m10ia_joint_1: type revolute, parent FANUC_m10ia_base_link, child FANUC_m10ia_link_1, origin xyz=0 0 0.450 rpy=0 0 0, axis 0 0 1, limit lower=-3.14 upper=3.14 effort=0 velocity=3.67
- added joint FANUC_m10ia_joint_2: type revolute, parent FANUC_m10ia_link_1, child FANUC_m10ia_link_2, origin xyz=0.150 0 0 rpy=0 0 0, axis 0 1 0, limit lower=-1.57 upper=2.79 effort=0 velocity=3.32
- added joint FANUC_m10ia_joint_3: type revolute, parent FANUC_m10ia_link_2, child FANUC_m10ia_link_3, origin xyz=0 0 0.600 rpy=0 0 0, axis 0 -1 0, limit lower=-3.14 upper=4.61 effort=0 velocity=3.67
- added joint FANUC_m10ia_joint_4: type revolute, parent FANUC_m10ia_link_3, child FANUC_m10ia_link_4, origin xyz=0 0 0.200 rpy=0 0 0, axis -1 0 0, limit lower=-3.31 upper=3.31 effort=0 velocity=6.98
- added joint FANUC_m10ia_joint_5: type revolute, parent FANUC_m10ia_link_4, child FANUC_m10ia_link_5, origin xyz=0.640 0 0 rpy=0 0 0, axis 0 -1 0, limit lower=-3.31 upper=3.31 effort=0 velocity=6.98
- added joint FANUC_m10ia_joint_6: type revolute, parent FANUC_m10ia_link_5, child FANUC_m10ia_link_6, origin xyz=0.100 0 0 rpy=0 0 0, axis -1 0 0, limit lower=-6.28 upper=6.28 effort=0 velocity=10.47
- added joint FANUC_m10ia_joint_6-tool0: type fixed, parent FANUC_m10ia_link_6, child FANUC_m10ia_tool, origin xyz=0 0 0 rpy=0 1.57079632679 0
- added joint FANUC_m10ia_pose: type fixed, parent world, child FANUC_m10ia_base_link, origin xyz=0 0.0 5.0 rpy=0.0 0.0 0.0
- joint curve_1_pose: origin xyz=0 0.0 5.0 rpy=0.0 0.0 0.0 -> xyz=0 2.0 0.0 rpy=0.0 0.0 0.0
- joint curve_2_pose: origin xyz=0 0.0 -5.0 rpy=0.0 0.0 0.0 -> xyz=0 -2.0 0.0 rpy=0.0 0.0 0.0
- joint joint_6-tool0: child tool0 -> ABB_6640_180_255_tool
