Commit message: curve 1 half get de result without collision (yaaaaaa!!)

File: config/urdf/fanuc_cell.urdf (robot description, URDF)
Before this commit: robot fanuc_cell, 22 links, 21 joints
Links:
- added link Ceiling; collision box size=1.8 1.7 0.01; visual box size=1.8 1.7 0.01
- added link Wall4; collision box size=1.8 0.01 1.3; visual box size=1.8 0.01 1.3
Joints:
- added joint Ceiling_pose: type fixed, parent world, child Ceiling, origin xyz=0.5 -0.27 1.45 rpy=0.0 0.0 0
- added joint Wall4_pose: type fixed, parent world, child Wall4, origin xyz=0.5 0.585 0.8 rpy=0.0 0.0 0

Commit message: run fanuc real robot test diffevo

File: config/urdf/fanuc_cell.urdf (robot description, URDF)
Before this commit: robot fanuc_cell, 24 links, 23 joints
Links:
- removed link Wall4
Joints:
- removed joint Wall4_pose
